Commit message: feat(mock_hardware): add high-fidelity Furuta pendulum mock plant and Raylib 3D visualizer
- Implement coupled 2-DOF Furuta Lagrangian dynamics matching physical CAD specs (L1, l2, m2, J1, J2)
- Implement realistic actuator and sensor models (stepper torque feasibility, step-loss modeling, cover travel markings, magnetic encoder quantization and filtering)
- Add standalone CAD-styled Raylib 3D visualizer running on an isolated thread with 4x MSAA anti-aliasing, studio palette, zero-overlap precision joint, locked framing (no zoom), non-flickering sim time card, and interactive disturbance injection
- Add integration test suite (test_mock_pendulum_launch.py) covering mock hardware activation, interface exports, and controller command claims
- Update CMakeLists.txt with WITH_RAYLIB option, auto-detection, and headless CI fallback
- Expose visualize launch argument in inverted_pendulum_mock.launch.py

File: demos/inverted_pendulum/inverted_pendulum_ros/urdf/inverted_pendulum_mock.urdf (robot description, URDF)
Before this commit: robot inverted_pendulum_mock, 3 links, 2 joints
Joints:
- joint pendulum_joint: origin xyz=0.2 0 0 rpy=0 0 0 -> xyz=0.062 0 0 rpy=0 0 0

Commit message: Revert "feat(inverted_pendulum): energy-shaping swing-up and full-state LQR b…"
This reverts commit 6cd225f79d563df848a6ed914afabb142eb42992.

File: demos/inverted_pendulum/inverted_pendulum_ros/urdf/inverted_pendulum_mock.urdf (robot description, URDF)
Before this commit: robot inverted_pendulum_mock, 3 links, 2 joints
Joints:
- joint pendulum_joint: origin xyz=0.062 0 0 rpy=0 0 0 -> xyz=0.2 0 0 rpy=0 0 0
